File: src/pcb/battery_pcb/Front_PCB.kicad_pcb (KiCad board)
At the start: 4 copper layers, 172.2 x 91.8 mm, 92 parts, among them IC1 TSYS01, IC2 TSYS01, J1 1778719, J10 464379206, J11 AMT0450003DB0000G, J2 1778719, J3 1778735, J4 AMT0450003DB0000G, J5 61300211121, J7 AMT0450003DB0000G, J8 AMT0450003DB0000G, J9 464379206, Q1 SIR804DP-T1-GE3, Q3 S400N08TL, Q4 S400N08TL, Q5 S400N08TL, Q6 S400N08TL, Q7 S400N08TL, Q8 TLP291_GB-TP,SE, Q9 SIR804DP-T1-GE3, U2 TSR_0.6-48120WI, U3 CPC1019N

Commit message: feat(pcb): replace PT3 Main PCB sources with Dev-Kit V1.2, battery PCB with V1.3
The Main PCB KiCad project on main was the PT3 first revision (September
2025). The Dev-Kit aircraft flies Main PCB V1.2 (January 2026), which moved
the payload and HV switching to MOSFETs driven by CPC1019N SSRs, added the
backup 5 V supply (U4), the dedicated lidar connector (U5), JST-GH
connectors, and the Raspberry Pi standoffs. Designators and control channels
differ between the two revisions, so documentation citing the old files was
wrong for the flying board.

main_pcb: V1.2 rounded project (board, schematic, four sub sheets, library
tables, EasyEDA library, production BOM, positions, IPC netlist and the
V1.2 fabrication zip). The stale netlist export (2025-06-02) and the PT3
fabrication zip are removed.

battery_pcb: Front PCB V1.3 project and STEP, with the V1.2 and V1.3
fabrication zips kept under production/.

fc_pcb and attach_pcb are unchanged.

Co-Authored-By: Claude Fable 5.1 <noreply@anthropic.com>
Parts:
- removed C2: 100nF, Capacitor_SMD:C_0805_2012Metric_Pad1.18x1.45mm_HandSolder
- removed IC2: TSYS01, Samacsys:QFN65P400X400X90-17N
- removed JP5, JP8: SolderJumper_2_Open, Snapeda:SolderJumper-2_P1.3mm_Open_RoundedPad1.0x1.5mm
- removed JP6: SolderJumper_2_Open, Snapeda:SolderJumper-2_P1.3mm_Bridged2Bar_RoundedPad1.0x1.5mm
- removed R11, R5, R6: 100k, Resistor_SMD:R_0805_2012Metric_Pad1.20x1.40mm_HandSolder
- added D10: ES3D, PCM_JLCPCB:D_SMC(DO-214AB), F.Cu at (107.1, 102.3)
- added D11: ES3D, PCM_JLCPCB:D_SMC(DO-214AB), F.Cu at (95.2, 116.6)
- added D3: ~, Snapeda:SMC_L6.9-W5.9-LS7.9-BI, B.Cu at (97.6, 119.9)
- Q1, Q9: value SIR804DP-T1-GE3 -> SIR570DP-T1-RE3; footprint Samacsys:SIR804DPT1GE3 -> EasyEDA_Lib:POWERPAK-SO-8_L5.9-W4.9-P1.27-LS6.2-BL
- Q8: value TLP291_GB-TP,SE -> CPC1019N; footprint Samacsys:SOIC127P700X230-4N -> Samacsys:SOP254P610X218-4N
- R14: value 420 -> 1K5
- R2: value 100k -> 0R
- R24, R27, R28, R29, R30, R31, R38: value 220K -> 10K
- moved R2 63.3 mm to (187.5, 88.3), turned to 90 degrees
- moved JP4 21.2 mm to (113.7, 106.6), turned to 0 degrees
- moved R4 21.0 mm to (110.1, 106.6), turned to 0 degrees
- moved JP3 19.0 mm to (115.3, 109.1), turned to 0 degrees
- moved IC1 18.8 mm to (132.8, 107.4)
- moved JP7 18.8 mm to (136.0, 111.4)
- moved C1 18.7 mm to (125.5, 107.5)
- moved R3 17.5 mm to (110.1, 109.1), turned to 0 degrees
- moved R10 16.5 mm to (130.0, 111.6)
- moved R1 16.3 mm to (129.3, 103.7), turned to 0 degrees
- moved R14 7.76 mm to (122.8, 97.5), turned to -90 degrees
- moved F4 3.17 mm to (97.7, 130.6), turned to 90 degrees
- moved Q8 0.60 mm to (115.3, 97.1)
- turned Q1 to 90 degrees
- turned Q9 to 90 degrees
Connections:
- F1 pad 2: Net-(Q1-S) -> Net-(F1-Pad2)
- F2 pad 1: Net-(Q9-S) -> Net-(F2-Pad1)
- J3 pad 1: /SSR_S -> /BYP_S
- J3 pad 2: +12V -> /SSR_S2
- J3 pad 3: +5V -> /SSR_S
- J3 pad 4: GND -> +12V
- J3 pad 5: unconnected-(J3-Pad5) -> +5V
- J3 pad 6: /BYP_S -> GND
- Q1 pad 1: Net-(Q1-G) -> Net-(F1-Pad2)
- Q1 pad 2: Net-(Q1-D) -> Net-(F1-Pad2)
- Q1 pad 3: Net-(Q1-S) -> Net-(F1-Pad2)
- Q9 pad 1: Net-(Q9-G) -> Net-(F2-Pad1)
- Q9 pad 2: /PW_- -> Net-(F2-Pad1)
- Q9 pad 3: Net-(Q9-S) -> Net-(F2-Pad1)
- R15 pad 1: Net-(Q1-D) -> Net-(D10-Pad2)
- R16 pad 1: Net-(Q1-D) -> Net-(D10-Pad2)
- R2 pad 1: +3V3 -> /SSR_S
- R2 pad 2: Net-(IC2-PS) -> /SSR_S2
Routing:
- net /SSR_S2: track 0.00 -> 79.4 mm, vias 0 -> 2
- net Net-(D10-Pad2): track 0.00 -> 67.2 mm, vias 0 -> 1
- net /BAT_+: track 58.0 -> 121.4 mm, vias 112 -> 113
- net Net-(Q1-D): track 50.8 -> 0.00 mm
- net +3V3: track 318.1 -> 269.7 mm, vias 5 -> 3
- net Net-(IC2-CSB): track 38.7 -> 0.00 mm, vias 2 -> 0
- net GND: track 63.8 -> 28.5 mm
- net Net-(Q1-S): track 32.1 -> 0.00 mm, vias 2 -> 0
- net Net-(F1-Pad2): track 0.00 -> 32.1 mm, vias 0 -> 2
- net Net-(IC2-PS): track 31.0 -> 0.00 mm, vias 2 -> 0
- net /I2C_SDA: track 206.1 -> 176.8 mm, vias 3 -> 2
- net /I2C_SCL: track 200.2 -> 171.7 mm
- net Net-(Q9-S): track 22.7 -> 0.00 mm, vias 1 -> 0
- net Net-(F2-Pad1): track 0.00 -> 22.2 mm, vias 0 -> 1
- net /SSR_S: track 83.4 -> 91.7 mm
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- added copper zone on B.Cu, net Net-(D10-Pad2)
- added copper zone on B.Cu, net Net-(F1-Pad2)
- added copper zone on B.Cu, net Net-(F2-Pad1)
- removed copper zone on B.Cu, net Net-(Q1-D)
- removed copper zone on B.Cu, net Net-(Q1-S)
- removed copper zone on B.Cu, net Net-(Q9-S)
Other:
- board text added: "ARROW Project Quiver BC_PCB V1.3 12/25"
- board text added: "BYP"
- board text added: "SSR"
- board text added: "SSR2"
- board text added: "SW+ SW- LED+ LED-"
- board text removed: "ARROW Project Quiver BC_PCB V1.2 09/25"
- board text removed: "BYP_S"
- board text removed: "LED+ LED- SW+ SW-"
- board text removed: "SSR_S"
- board text removed: "X"
