File: src/pcb/battery_pcb/Front_PCB.kicad_sch (KiCad schematic)
At the start: 92 parts, among them IC1 TSYS01, IC2 TSYS01, J1 1778719, J10 464379206, J11 AMT0450003DB0000G, J2 1778719, J3 1778735, J4 AMT0450003DB0000G, J5 61300211121, J7 AMT0450003DB0000G, J8 AMT0450003DB0000G, J9 464379206, Q1 SIR804DP-T1-GE3, Q3 S400N08TL, Q4 S400N08TL, Q5 S400N08TL, Q6 S400N08TL, Q7 S400N08TL, Q8 TLP291_GB-TP,SE, Q9 SIR804DP-T1-GE3, U2 TSR_0.6-48120WI, U3 CPC1019N

Commit message: feat(pcb): replace PT3 Main PCB sources with Dev-Kit V1.2, battery PCB with V1.3
The Main PCB KiCad project on main was the PT3 first revision (September
2025). The Dev-Kit aircraft flies Main PCB V1.2 (January 2026), which moved
the payload and HV switching to MOSFETs driven by CPC1019N SSRs, added the
backup 5 V supply (U4), the dedicated lidar connector (U5), JST-GH
connectors, and the Raspberry Pi standoffs. Designators and control channels
differ between the two revisions, so documentation citing the old files was
wrong for the flying board.

main_pcb: V1.2 rounded project (board, schematic, four sub sheets, library
tables, EasyEDA library, production BOM, positions, IPC netlist and the
V1.2 fabrication zip). The stale netlist export (2025-06-02) and the PT3
fabrication zip are removed.

battery_pcb: Front PCB V1.3 project and STEP, with the V1.2 and V1.3
fabrication zips kept under production/.

fc_pcb and attach_pcb are unchanged.

Co-Authored-By: Claude Fable 5.1 <noreply@anthropic.com>
Parts:
- removed C2: 100nF, Capacitor_SMD:C_0805_2012Metric_Pad1.18x1.45mm_HandSolder, symbol Device:C
- removed IC2: TSYS01, Samacsys:QFN65P400X400X90-17N, symbol Samacsys_kicad_sym:TSYS01
- removed JP5, JP8: SolderJumper_2_Open, Snapeda:SolderJumper-2_P1.3mm_Open_RoundedPad1.0x1.5mm, symbol Jumper:SolderJumper_2_Open
- removed JP6: SolderJumper_2_Open, Snapeda:SolderJumper-2_P1.3mm_Bridged2Bar_RoundedPad1.0x1.5mm, symbol Jumper:SolderJumper_2_Bridged
- removed R11, R5, R6: 100k, Resistor_SMD:R_0805_2012Metric_Pad1.20x1.40mm_HandSolder, symbol Device:R
- added D10, D11: ES3D, PCM_JLCPCB:D_SMC(DO-214AB), symbol Snapeda:ES3D_C241735
- added D3: ~, Snapeda:SMC_L6.9-W5.9-LS7.9-BI, symbol EasyEDA_Lib:SMCJ75CA_C310078
- Q1, Q9: value SIR804DP-T1-GE3 -> SIR570DP-T1-RE3; footprint Samacsys:SIR804DPT1GE3 -> EasyEDA_Lib:POWERPAK-SO-8_L5.9-W4.9-P1.27-LS6.2-BL; symbol Samacsys_kicad_sym:SIR804DP-T1-GE3 -> Snapeda:SIR570DP-T1-RE3; LCSC Part Name (none) -> 1个N沟道 耐压:150V 电流:77.4A; Manufacturer (none) -> VISHAY(威世); Manufacturer Part (none) -> SIR570DP-T1-RE3; Supplier (none) -> LCSC; Supplier Part (none) -> C3279563
- Q8: value TLP291_GB-TP,SE -> CPC1019N; footprint Samacsys:SOIC127P700X230-4N -> Samacsys:SOP254P610X218-4N; symbol Samacsys_kicad_sym:TLP291_GB-TP,SE -> Samacsys:CPC1019N; Height 2.3 -> 2.184; Manufacturer_Name Toshiba -> LITTELFUSE; Manufacturer_Part_Number TLP291(GB-TP,SE -> CPC1019N; Mouser Part Number 757-TLP291GB-TPSE -> 849-CPC1019N; Mouser Price/Stock https://www.mouser.co.uk/ProductDetail/Toshiba/TLP291GB-TPS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 -> https://www.mouser.co.uk/ProductDetail/IXYS-Integrated-Circ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
- R14: value 420 -> 1K5
- R2: value 100k -> 0R
- R24, R27, R28, R29, R30, R31, R38: value 220K -> 10K
Connections:
- net +12V: now also J3.4; no longer J3.2
- net +3V3: no longer R2.1
- net +5V: now also J3.5; no longer J3.3
- net BAT_+: now also D10.1, D11.1
- net BAT_-: now also D3.1 (K)
- net BYP_S: now also J3.1; no longer J3.6
- net GND: now also J3.6; no longer J3.4
- net PW_-: now also Q9.5 (D), Q9.6 (D), Q9.7 (D), Q9.8 (D), D11.2, D3.2 (A); no longer Q9.2 (D)
- net SSR_S: now also J3.3, R2.1; no longer J3.1
- net at R15.1, R16.1: now also Q1.5 (D), Q1.6 (D), Q1.7 (D), Q1.8 (D), D10.2; no longer Q1.2 (D)
- net SSR_S2: now reaches R2.2
- net SSR_S2: now also J3.2
- net at D1.2, R18.2, R24.1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: now also Q1.4 (G); no longer Q1.1 (G)
- net at D9.2, R37.2, R38.1: now also Q9.4 (G); no longer Q9.1 (G)
- net at F2.1, Q9.3 (S): now also Q9.1 (S), Q9.2 (S)
- net at F1.2, Q1.3 (S): now also Q1.1 (S), Q1.2 (S)
- no-connect marks 21 -> 11
Other:
- note added: "Temperature sensor"
- note removed: "Temperature sensor 1 for precharge resistor"
- note removed: "Temperature sensor 2 for SSR mosfets"
- moved on the sheet: C1, IC1, J3, JP3, JP4, JP7, Q8, R1, R10, R12, R13, R15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
