File: src/pcb/main_pcb/CAN circuit.kicad_sch (KiCad schematic)
At the start: 17 parts, among them U1 TJA1049T/3J, U2 MCP2515-I/SO, X1 16MHz

Commit message: feat(pcb): replace PT3 Main PCB sources with Dev-Kit V1.2, battery PCB with V1.3
The Main PCB KiCad project on main was the PT3 first revision (September
2025). The Dev-Kit aircraft flies Main PCB V1.2 (January 2026), which moved
the payload and HV switching to MOSFETs driven by CPC1019N SSRs, added the
backup 5 V supply (U4), the dedicated lidar connector (U5), JST-GH
connectors, and the Raspberry Pi standoffs. Designators and control channels
differ between the two revisions, so documentation citing the old files was
wrong for the flying board.

main_pcb: V1.2 rounded project (board, schematic, four sub sheets, library
tables, EasyEDA library, production BOM, positions, IPC netlist and the
V1.2 fabrication zip). The stale netlist export (2025-06-02) and the PT3
fabrication zip are removed.

battery_pcb: Front PCB V1.3 project and STEP, with the V1.2 and V1.3
fabrication zips kept under production/.

fc_pcb and attach_pcb are unchanged.

Co-Authored-By: Claude Fable 5.1 <noreply@anthropic.com>
Parts:
- X1: footprint Samacsys:NX3225GD-STD-CRA-3 -> Samacsys:NX3225GB-16M-STD-CRA-2
Changed lines of the file:
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@@
 			)
 		)
-		(property "Footprint" "Samacsys:NX3225GD-STD-CRA-3"
+		(property "Footprint" "Samacsys:NX3225GB-16M-STD-CRA-2"
 			(at 178.232 116.84 0)
 			(effects
