File: src/pcb/main_pcb/ETHERNET.kicad_sch (KiCad schematic)
At the start: 4 parts, among them J47 GIGABLOX_NANO_SWITCH_REVA_MOD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, J48 SM04B-GHS-TB_LF__SN_, J51 GIGABLOX_NANO_SWITCH_REVA_MOD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, J52 SM04B-GHS-TB_LF__SN_

Commit message: feat(pcb): replace PT3 Main PCB sources with Dev-Kit V1.2, battery PCB with V1.3
The Main PCB KiCad project on main was the PT3 first revision (September
2025). The Dev-Kit aircraft flies Main PCB V1.2 (January 2026), which moved
the payload and HV switching to MOSFETs driven by CPC1019N SSRs, added the
backup 5 V supply (U4), the dedicated lidar connector (U5), JST-GH
connectors, and the Raspberry Pi standoffs. Designators and control channels
differ between the two revisions, so documentation citing the old files was
wrong for the flying board.

main_pcb: V1.2 rounded project (board, schematic, four sub sheets, library
tables, EasyEDA library, production BOM, positions, IPC netlist and the
V1.2 fabrication zip). The stale netlist export (2025-06-02) and the PT3
fabrication zip are removed.

battery_pcb: Front PCB V1.3 project and STEP, with the V1.2 and V1.3
fabrication zips kept under production/.

fc_pcb and attach_pcb are unchanged.

Co-Authored-By: Claude Fable 5.1 <noreply@anthropic.com>
Parts:
- added U13, U14, U15, U16: SMTWEM245STR, Snapeda:SCREW-SMD_BD4.4-D2.8-H4.5, symbol Snapeda:SMTWEM245STR
Connections:
- no-connect marks 32 -> 30
